Commit message: Features commits 	- Se agrego codigo de la placa arduino 	- Se actaulizo modelado hermes 3 (faltan colores al modelo): 		- Para simulacion en gazebo quedo el modelo hermes 2 		- Para visualizacion unicamente de cuando mapeamos quedo el modelo del hermes 3 	- Se modifico parametros de mapeo para mejorar el mismo (verificar que funcionen)

File: src/hermesIII/model/urdf/modelo_HermesII.urdf (robot description, URDF)
Before this commit: robot HermesIII, 37 links, 36 joints
Links:
- link base_link: geometry collision mesh filename=package://hermesIII/model/dae/Base.dae; visual mesh filename=package://hermesIII/model/dae/Base.dae
- link cylinderE_wheel_back_link: geometry collision mesh filename=package://hermesIII/model/dae/Cilindro.dae; visual mesh filename=package://hermesIII/model/dae/Cilindro.dae
- link cylinderE_wheel_front_link: geometry collision mesh filename=package://hermesIII/model/dae/Cilindro.dae; visual mesh filename=package://hermesIII/model/dae/Cilindro.dae
- link cylinderE_wheel_left_link: geometry collision mesh filename=package://hermesIII/model/dae/Cilindro.dae; visual mesh filename=package://hermesIII/model/dae/Cilindro.dae
- link cylinderE_wheel_right_link: geometry collision mesh filename=package://hermesIII/model/dae/Cilindro.dae; visual mesh filename=package://hermesIII/model/dae/Cilindro.dae
- link cylinderNE_wheel_back_link: geometry collision mesh filename=package://hermesIII/model/dae/Cilindro.dae; visual mesh filename=package://hermesIII/model/dae/Cilindro.dae
- link cylinderNE_wheel_front_link: geometry collision mesh filename=package://hermesIII/model/dae/Cilindro.dae; visual mesh filename=package://hermesIII/model/dae/Cilindro.dae
- link cylinderNE_wheel_left_link: geometry collision mesh filename=package://hermesIII/model/dae/Cilindro.dae; visual mesh filename=package://hermesIII/model/dae/Cilindro.dae
- link cylinderNE_wheel_right_link: geometry collision mesh filename=package://hermesIII/model/dae/Cilindro.dae; visual mesh filename=package://hermesIII/model/dae/Cilindro.dae
- link cylinderNO_wheel_back_link: geometry collision mesh filename=package://hermesIII/model/dae/Cilindro.dae; visual mesh filename=package://hermesIII/model/dae/Cilindro.dae
- link cylinderNO_wheel_front_link: geometry collision mesh filename=package://hermesIII/model/dae/Cilindro.dae; visual mesh filename=package://hermesIII/model/dae/Cilindro.dae
- link cylinderNO_wheel_left_link: geometry collision mesh filename=package://hermesIII/model/dae/Cilindro.dae; visual mesh filename=package://hermesIII/model/dae/Cilindro.dae
- link cylinderNO_wheel_right_link: geometry collision mesh filename=package://hermesIII/model/dae/Cilindro.dae; visual mesh filename=package://hermesIII/model/dae/Cilindro.dae
- link cylinderN_wheel_back_link: geometry collision mesh filename=package://hermesIII/model/dae/Cilindro.dae; visual mesh filename=package://hermesIII/model/dae/Cilindro.dae
- link cylinderN_wheel_front_link: geometry collision mesh filename=package://hermesIII/model/dae/Cilindro.dae; visual mesh filename=package://hermesIII/model/dae/Cilindro.dae
- link cylinderN_wheel_left_link: geometry collision mesh filename=package://hermesIII/model/dae/Cilindro.dae; visual mesh filename=package://hermesIII/model/dae/Cilindro.dae
- link cylinderN_wheel_right_link: geometry collision mesh filename=package://hermesIII/model/dae/Cilindro.dae; visual mesh filename=package://hermesIII/model/dae/Cilindro.dae
- link cylinderO_wheel_back_link: geometry collision mesh filename=package://hermesIII/model/dae/Cilindro.dae; visual mesh filename=package://hermesIII/model/dae/Cilindro.dae
- link cylinderO_wheel_front_link: geometry collision mesh filename=package://hermesIII/model/dae/Cilindro.dae; visual mesh filename=package://hermesIII/model/dae/Cilindro.dae
- link cylinderO_wheel_left_link: geometry collision mesh filename=package://hermesIII/model/dae/Cilindro.dae; visual mesh filename=package://hermesIII/model/dae/Cilindro.dae
- link cylinderO_wheel_right_link: geometry collision mesh filename=package://hermesIII/model/dae/Cilindro.dae; visual mesh filename=package://hermesIII/model/dae/Cilindro.dae
- link cylinderSE_wheel_back_link: geometry collision mesh filename=package://hermesIII/model/dae/Cilindro.dae; visual mesh filename=package://hermesIII/model/dae/Cilindro.dae
- link cylinderSE_wheel_front_link: geometry collision mesh filename=package://hermesIII/model/dae/Cilindro.dae; visual mesh filename=package://hermesIII/model/dae/Cilindro.dae
- link cylinderSE_wheel_left_link: geometry collision mesh filename=package://hermesIII/model/dae/Cilindro.dae; visual mesh filename=package://hermesIII/model/dae/Cilindro.dae
- link cylinderSE_wheel_right_link: geometry collision mesh filename=package://hermesIII/model/dae/Cilindro.dae; visual mesh filename=package://hermesIII/model/dae/Cilindro.dae
- link cylinderSO_wheel_back_link: geometry collision mesh filename=package://hermesIII/model/dae/Cilindro.dae; visual mesh filename=package://hermesIII/model/dae/Cilindro.dae
- link cylinderSO_wheel_front_link: geometry collision mesh filename=package://hermesIII/model/dae/Cilindro.dae; visual mesh filename=package://hermesIII/model/dae/Cilindro.dae
- link cylinderSO_wheel_left_link: geometry collision mesh filename=package://hermesIII/model/dae/Cilindro.dae; visual mesh filename=package://hermesIII/model/dae/Cilindro.dae
- link cylinderSO_wheel_right_link: geometry collision mesh filename=package://hermesIII/model/dae/Cilindro.dae; visual mesh filename=package://hermesIII/model/dae/Cilindro.dae
- link cylinderS_wheel_back_link: geometry collision mesh filename=package://hermesIII/model/dae/Cilindro.dae; visual mesh filename=package://hermesIII/model/dae/Cilindro.dae
- link cylinderS_wheel_front_link: geometry collision mesh filename=package://hermesIII/model/dae/Cilindro.dae; visual mesh filename=package://hermesIII/model/dae/Cilindro.dae
- link cylinderS_wheel_left_link: geometry collision mesh filename=package://hermesIII/model/dae/Cilindro.dae; visual mesh filename=package://hermesIII/model/dae/Cilindro.dae
- link cylinderS_wheel_right_link: geometry collision mesh filename=package://hermesIII/model/dae/Cilindro.dae; visual mesh filename=package://hermesIII/model/dae/Cilindro.dae
- link wheel_back_link: geometry collision mesh filename=package://hermesIII/model/dae/wheel.dae; visual mesh filename=package://hermesIII/model/dae/wheel.dae
- link wheel_front_link: geometry collision mesh filename=package://hermesIII/model/dae/wheel.dae; visual mesh filename=package://hermesIII/model/dae/wheel.dae
- link wheel_left_link: geometry collision mesh filename=package://hermesIII/model/dae/wheel.dae; visual mesh filename=package://hermesIII/model/dae/wheel.dae
- link wheel_right_link: geometry collision mesh filename=package://hermesIII/model/dae/wheel.dae; visual mesh filename=package://hermesIII/model/dae/wheel.dae

File: src/hermesIII/model/urdf/modelo_HermesIII.urdf (robot description, URDF)
Before this commit: robot HermesIII, 37 links, 36 joints
Links:
- removed link cylinderE_wheel_back_link
- removed link cylinderE_wheel_front_link
- removed link cylinderE_wheel_left_link
- removed link cylinderE_wheel_right_link
- removed link cylinderNE_wheel_back_link
- removed link cylinderNE_wheel_front_link
- removed link cylinderNE_wheel_left_link
- removed link cylinderNE_wheel_right_link
- removed link cylinderNO_wheel_back_link
- removed link cylinderNO_wheel_front_link
- removed link cylinderNO_wheel_left_link
- removed link cylinderNO_wheel_right_link
- removed link cylinderN_wheel_back_link
- removed link cylinderN_wheel_front_link
- removed link cylinderN_wheel_left_link
- removed link cylinderN_wheel_right_link
- removed link cylinderO_wheel_back_link
- removed link cylinderO_wheel_front_link
- removed link cylinderO_wheel_left_link
- removed link cylinderO_wheel_right_link
- removed link cylinderSE_wheel_back_link
- removed link cylinderSE_wheel_front_link
- removed link cylinderSE_wheel_left_link
- removed link cylinderSE_wheel_right_link
- removed link cylinderSO_wheel_back_link
- removed link cylinderSO_wheel_front_link
- removed link cylinderSO_wheel_left_link
- removed link cylinderSO_wheel_right_link
- removed link cylinderS_wheel_back_link
- removed link cylinderS_wheel_front_link
- removed link cylinderS_wheel_left_link
- removed link cylinderS_wheel_right_link
- removed link wheel_back_link
- removed link wheel_front_link
- removed link wheel_left_link
- removed link wheel_right_link
- link base_link: mass 1.0 -> None; geometry visual mesh filename=package://hermesIII/model/dae/Hermes3_2017.dae scale=0.2 0.2 0.2
Joints:
- removed joint base_to_back_wheel
- removed joint base_to_front_wheel
- removed joint base_to_left_wheel
- removed joint base_to_right_wheel
- removed joint cylinderE_to_back_wheel
- removed joint cylinderE_to_front_wheel
- removed joint cylinderE_to_left_wheel
- removed joint cylinderE_to_right_wheel
- removed joint cylinderNE_to_back_wheel
- removed joint cylinderNE_to_front_wheel
- removed joint cylinderNE_to_left_wheel
- removed joint cylinderNE_to_right_wheel
- removed joint cylinderNO_to_back_wheel
- removed joint cylinderNO_to_front_wheel
- removed joint cylinderNO_to_left_wheel
- removed joint cylinderNO_to_right_wheel
- removed joint cylinderN_to_back_wheel
- removed joint cylinderN_to_front_wheel
- removed joint cylinderN_to_left_wheel
- removed joint cylinderN_to_right_wheel
- removed joint cylinderO_to_back_wheel
- removed joint cylinderO_to_front_wheel
- removed joint cylinderO_to_left_wheel
- removed joint cylinderO_to_right_wheel
- removed joint cylinderSE_to_back_wheel
- removed joint cylinderSE_to_front_wheel
- removed joint cylinderSE_to_left_wheel
- removed joint cylinderSE_to_right_wheel
- removed joint cylinderSO_to_back_wheel
- removed joint cylinderSO_to_front_wheel
- removed joint cylinderSO_to_left_wheel
- removed joint cylinderSO_to_right_wheel
- removed joint cylinderS_to_back_wheel
- removed joint cylinderS_to_front_wheel
- removed joint cylinderS_to_left_wheel
- removed joint cylinderS_to_right_wheel
